File: mainboard/AddressDecoding.kicad_sch (KiCad schematic)
At the start: 15 parts, among them SW1 RAM Size, U5 74LS138, U6 74LS03, U7 74LS08, U8 74LS138, U9 74LS32

Commit message: layout work
Connections:
- no-connect marks 1 -> 2
Changed lines of the file:
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@@
+	)
+	(no_connect
+		(at 181.61 72.39)
 	)
 	(no_connect
