File: mainboard/Console.kicad_pcb (KiCad board)
At the start: 2 copper layers, 244 x 244 mm, 261 parts, among them J10 Joystick, J11 Keyboard, J13 I/O Port, J15 GROM Port, J16 Rom Select 1, J17 Rom Select 2, J18 Cassette, J2 Power LED, J4 UNICORN PORT, J5 ROM Select, J6 ROM Select, J7 Sound Clock Select, J8 AUDIO OUT, J9 VIDEO OUT, P1 CONN_1, P10 CONN_1, P11 CONN_1, P12 CONN_1, P13 CONN_10X2, P14 POWER_SW, P2 CONN_1, P3 CONN_1, P4 CONN_1, P5 CONN_1, P6 CONN_1, P7 CONN_1, P8 CONN_1, P9 CONN_1, Q1 TIS92, Q2 2N3904, Q3 2N4946 or TIS92, Q4 2N4946 or TIS92, SW1 RAM Size, SW2 Internal Cart ROM Enable, SW3 POWER, U1 TIM9904, U10 74LS00, U11 74LS244, U12 74LS373, U13 74LS245, U14 74LS00, U15 74LS04, U16 74LS74, U17 74LS194, U18 74LS00, U19 LM2901, U2 TMS9900, U21 LM2903, U22 74LS04, U23 74HCT14, U24 74LS04, U25 74LS74, U26 TMC0430, U27 TMC0430, U28 TMC0430, U29 HM62256BLP, U3 74LS04, U30 HM62256BLP, U31 27C64, U32 27C64, U33 SN76489, U34 TMS9918, U35 74LS574, U36 74LS574, U37 HM62256BLP, U38 74LS574, U39 TMS9901, U4 74LS32, U40 74LS156, U41 74LS244, U42 74LS367, U43 74LS367, U44 74LS379, U45 27C010-C, U46 RC4558, U47 74LS06, U48 TIL119, U49 TIL119, U5 74LS138, U6 74LS03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

Commit message: layout work
Parts:
- removed U43: 74LS367, Custom:STD_DDW_DIP16
- added J1: Conn_02x30_Odd_Even, Custom:STD_DDW_CARDEDGE60, F.Cu at (51.2, 115.4)
- added J12: Conn_02x30_Odd_Even, Custom:STD_DDW_CARDEDGE60, F.Cu at (88.4, 115.3)
- added J14: Conn_02x30_Odd_Even, Custom:STD_DDW_CARDEDGE60, F.Cu at (107.1, 115.1)
- added J19: Screw_Terminal_01x05, TerminalBlock_RND:TerminalBlock_RND_205-00004_1x05_P5.00mm_Horizontal, F.Cu at (37.3, 246.4)
- added J3: Conn_02x30_Odd_Even, Custom:STD_DDW_CARDEDGE60, F.Cu at (69.8, 115.5)
- added R81: 4.7kΩ, Custom:STD_DDW_RESISTOR, F.Cu at (107.3, 207.7)
- added R82: 100Ω, Custom:STD_DDW_RESISTOR, F.Cu at (107.3, 211.7)
- added R83: 4.7kΩ, Custom:STD_DDW_RESISTOR, F.Cu at (107.3, 215.8)
- added R84: 330Ω, Custom:STD_DDW_RESISTOR, F.Cu at (107.3, 219.8)
- added U20: 74LS244, Custom:STD_DDW_DIP20, F.Cu at (42.0, 214.1)
- added U50: 74LS245, Custom:STD_DDW_DIP20, F.Cu at (59.2, 214.9)
- J13: value I/O Port -> Conn_02x30_Odd_Even; footprint Custom:STD_DDW_CARDEDGE_44 -> Custom:STD_DDW_CARDEDGE60
- R49: value 100Ω -> 330Ω
- R52, R53: value 4.7kΩ -> 330Ω
- R54: value 100Ω -> 4.7kΩ
- U42: value 74LS367 -> 74LS244; footprint Custom:STD_DDW_DIP16 -> Custom:STD_DDW_DIP20
- moved J13 309.3 mm to (32.5, 115.4), turned to 90 degrees
- moved CR4 102.8 mm to (84.2, 220.7)
- moved R56 92.5 mm to (81.3, 200.8)
- moved R64 91.4 mm to (81.3, 213.5)
- moved C60 83.3 mm to (199.2, 61.1)
- moved R63 80.3 mm to (81.7, 207.1)
- moved C10 55.3 mm to (109.5, 199.4)
- moved R10 55.3 mm to (114.7, 69.7)
- moved R49 54.9 mm to (116.1, 56.6)
- moved U46 54.4 mm to (99.0, 191.0)
- moved R52 38.9 mm to (134.7, 82.3)
- moved R9 38.3 mm to (124.0, 81.9)
- moved C27 6.46 mm to (115.5, 62.8)
Connections:
- J13 pad 1: +5V -> +8V
- J13 pad 10: IO_A3 -> IO_SNDIN
- J13 pad 11: IO_A12 -> RDBENA
- J13 pad 12: READY_~{HOLD} -> IO_HIGH
- J13 pad 13: /GROM-IO-Port/~{IO_LOAD} -> IO_HIGH
- J13 pad 15: IO_A13 -> IO_HIGH
- J13 pad 16: IO_A14 -> IO_HIGH
- J13 pad 17: IO_A7 -> EXTINT
- J13 pad 18: IO_A9 -> unconnected-(J13-Pin_18-Pad18)
- J13 pad 19: IO_A15-CRUOUT -> IO_D7
- J13 pad 2: SBE -> +8V
- J13 pad 20: IO_A2 -> GND
- J13 pad 21: GND -> IO_D5
- J13 pad 22: /GROM-IO-Port/~{IO_CRUCLK} -> IO_D6
- J13 pad 23: GND -> IO_D3
- J13 pad 24: /GROM-IO-Port/IO_Ø3 -> IO_D4
- J13 pad 25: GND -> IO_D1
- J13 pad 26: /GROM-IO-Port/~{IO_WE} -> IO_D2
- J13 pad 28: /GROM-IO-Port/~{IO_MBE} -> IO_D0
- J13 pad 29: IO_A6 -> IO_A14
- J13 pad 30: IO_A1 -> IO_A15-CRUOUT
- J13 pad 31: IO_A0 -> IO_A12
- J13 pad 32: ~{MEMEN} -> IO_A13
- J13 pad 33: /GROM-IO-Port/IO_CRUIN -> IO_A10
- J13 pad 34: D7 -> IO_A11
- J13 pad 35: D4 -> IO_A8
- J13 pad 36: D6 -> IO_A9
- J13 pad 37: D0 -> IO_A6
- J13 pad 38: D5 -> IO_A7
- J13 pad 39: D2 -> IO_A4
- J13 pad 4: /GROM-IO-Port/~{IO_EXT_INT} -> IO_READY_~{HOLD}
- J13 pad 40: D1 -> IO_A5
- J13 pad 41: /GROM-IO-Port/HOLD/IAQ -> IO_A2
- J13 pad 42: D3 -> IO_A3
- J13 pad 43: -5V -> IO_A0
- J13 pad 44: IO_SNDIN -> IO_A1
- J13 pad 5: IO_A5 -> GND
- J13 pad 6: IO_A10 -> ~{IO_RESET}
- J13 pad 7: IO_A4 -> GND
- J13 pad 8: IO_A11 -> unconnected-(J13-Pin_8-Pad8)
- J13 pad 9: /GROM-IO-Port/IO_DBIN -> unconnected-(J13-Pin_9-Pad9)
- R41 pad 1: /GROM-IO-Port/IO_Ø3 -> IO_Ø3
- R42 pad 1: /GROM-IO-Port/~{IO_WE} -> ~{IO_WE}
- R44 pad 1: /GROM-IO-Port/~{IO_CRUCLK} -> ~{IO_CRUCLK}
- R49 pad 1: /GROM-IO-Port/~{IO_LOAD} -> IO_SNDIN
- R49 pad 2: ~{LOAD} -> SNDIN
- R51 pad 2: /GROM-IO-Port/IO_CRUIN -> Net-(U42-O1b)
- R52 pad 1: +5V -> IO_SNDIN
- R52 pad 2: /GROM-IO-Port/~{IO_LOAD} -> SNDIN
- R53 pad 1: +5V -> IO_SNDIN
- R53 pad 2: /GROM-IO-Port/~{IO_EXT_INT} -> SNDIN
- R54 pad 1: /GROM-IO-Port/~{IO_EXT_INT} -> +5V
- R54 pad 2: EXTINT -> ~{IO_EXT_INT}
- R56 pad 2: /GROM-IO-Port/HOLD/IAQ -> HOLD/IAQ
- U22 pad 6: /GROM-IO-Port/~{IO_RESET} -> ~{IO_RESET}
- U22 pad 8: /GROM-IO-Port/IO_DBIN -> IO_DBIN
- U41 pad 3: /GROM-IO-Port/~{IO_MBE} -> ~{IO_MBE}
- U42 pad 10: A8 -> GND
- U42 pad 11: IO_A9 -> ~{MEMEN}
- U42 pad 12: A9 -> IO_A10
- U42 pad 13: IO_A14 -> IO_CRUIN
- U42 pad 14: A14 -> IO_A11
- U42 pad 15: GND -> EXTINT
- U42 pad 16: +5V -> IO_A12
- U42 pad 2: A13 -> A3
- U42 pad 3: IO_A13 -> IO_READY_~{HOLD}
- U42 pad 4: A7 -> A12
- U42 pad 5: IO_A7 -> ~{IO_EXT_INT}
- U42 pad 6: A6 -> A11
- U42 pad 7: IO_A6 -> Net-(U42-O1b)
- U42 pad 8: GND -> A10
- U42 pad 9: IO_A8 -> IO_~{MEMEN}
Other:
- board text added: "VERIFY CARD SPACING (VERT/HORIZ) FIX SCREENPRINT FIX ALIGNMENT FIX GROM SPACING ADD GROUND TO SCREW TERMINALS MOVE KEYBOARD CONNECTOR ADD RCA FOR SOUND AND VIDEO"

Commit message: layout work
Parts:
- removed J14: Conn_02x30_Odd_Even, Custom:STD_DDW_CARDEDGE60
- removed R84: 330Ω, Custom:STD_DDW_RESISTOR
- moved C70 54.9 mm to (81.0, 194.6)
- moved R58 49.9 mm to (96.8, 219.6)
- moved R59 49.8 mm to (96.8, 213.3)
- moved R60 49.8 mm to (96.8, 207.0)
- moved J19 20.6 mm to (57.4, 242.0), turned to 180 degrees
- moved J12 19.5 mm to (105.1, 125.4)
- moved J3 14.3 mm to (80.1, 125.4)
- moved J1 10.8 mm to (55.1, 125.4)
- moved J13 10.2 mm to (30.1, 125.4)
- moved C11 5.32 mm to (159.1, 182.8)
- moved R83 3.96 mm to (108.1, 219.6)
- moved R26 3.21 mm to (272.4, 63.4)
- moved C9 3.13 mm to (159.2, 172.9)
- moved C8 2.99 mm to (128.6, 156.9)
- moved U46 2.41 mm to (96.9, 190.0)
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Other:
- board text added: "VERIFY CARD SPACING (VERT/HORIZ) FIX SCREENPRINT FIX ALIGNMENT FIX GROM SPACING ADD GROUND TO SCREW TERMINALS MOVE KEYBOARD CONNECTOR ADD RCA FOR SOUND AND VIDEO ADD TIPI Connector"
- board text removed: "VERIFY CARD SPACING (VERT/HORIZ) FIX SCREENPRINT FIX ALIGNMENT FIX GROM SPACING ADD GROUND TO SCREW TERMINALS MOVE KEYBOARD CONNECTOR ADD RCA FOR SOUND AND VIDEO"

Commit message: layout work
Parts:
- removed J8: AUDIO OUT, Custom:STD_DDW_PINHEAD_V_1x02
- added J14: Conn_Coaxial, Custom:CUI_RCJ-047, F.Cu at (183.6, 19.3)
- J19: value Screw_Terminal_01x05 -> Screw_Terminal_01x06; footprint TerminalBlock_RND:TerminalBlock_RND_205-00004_1x05_P5.00mm_Horizontal -> TerminalBlock_RND:TerminalBlock_RND_205-00005_1x06_P5.00mm_Horizontal
- J9: value VIDEO OUT -> Conn_Coaxial; footprint Custom:STD_DDW_PINHEAD_V_1x02 -> Custom:CUI_RCJ-047
- moved R40 49.2 mm to (196.9, 75.2)
- moved C66 41.9 mm to (234.9, 46.6)
- moved R33 36.8 mm to (196.8, 68.8)
- moved R30 26.6 mm to (222.8, 46.9)
- moved J9 18.4 mm to (198.9, 19.2), turned to 90 degrees
- moved R31 17.1 mm to (175.2, 34.5), turned to 90 degrees
- moved J13 15.7 mm to (30.0, 141.0)
- moved J1 15.6 mm to (55.1, 141.0)
- moved J12 15.6 mm to (105.1, 141.0)
- moved J3 15.6 mm to (80.1, 141.0)
- moved C22 11.8 mm to (65.4, 233.2)
- moved C36 11.5 mm to (161.0, 21.8)
- moved C61 4.87 mm to (185.0, 35.4)
- moved Q2 3.42 mm to (190.2, 42.6)
- moved J19 2.71 mm to (60.1, 242.0)
Connections:
- J9 pad 2: /Video/COMVID -> SNDOUT
Other:
- board text removed: "VERIFY CARD SPACING (VERT/HORIZ) FIX SCREENPRINT FIX ALIGNMENT FIX GROM SPACING ADD GROUND TO SCREW TERMINALS MOVE KEYBOARD CONNECTOR ADD RCA FOR SOUND AND VIDEO ADD TIPI Connector"
