File: mainboard/Power.kicad_sch (KiCad schematic)
At the start: 82 parts, among them J2 Power LED, P1 CONN_1, P10 CONN_1, P11 CONN_1, P12 CONN_1, P13 CONN_10X2, P14 POWER_SW, P2 CONN_1, P3 CONN_1, P4 CONN_1, P5 CONN_1, P6 CONN_1, P7 CONN_1, P8 CONN_1, P9 CONN_1, SW3 POWER, U10 74LS00, U14 74LS00, U15 74LS04, U16 74LS74, U18 74LS00, U19 LM2901, U21 LM2903, U22 74LS04, U23 74HCT14, U24 74LS04, U25 74LS74, U3 74LS04, U4 74LS32, U46 RC4558, U47 74LS06, U6 74LS03, U7 74LS08, U9 74LS32

Commit message: layout work
Parts:
- added J19: Screw_Terminal_01x05, TerminalBlock_RND:TerminalBlock_RND_205-00004_1x05_P5.00mm_Horizontal, symbol Connector:Screw_Terminal_01x05
Connections:
- net +12V: now also J19.3 (Pin_3)
- net -12V: now also J19.4 (Pin_4)
- new net +15V: J19.2 (Pin_2)
- new net +8V: J19.1 (Pin_1)
- new net -15V: J19.5 (Pin_5)
Other:
- moved on the sheet: C76, C77, D2, D3, P13, P14, R78, R79, R80, SW3, U23A, U23B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

Commit message: layout work
Parts:
- J19: value Screw_Terminal_01x05 -> Screw_Terminal_01x06; footprint TerminalBlock_RND:TerminalBlock_RND_205-00004_1x05_P5.00mm_Horizontal -> TerminalBlock_RND:TerminalBlock_RND_205-00005_1x06_P5.00mm_Horizontal; symbol Connector:Screw_Terminal_01x05 -> Connector:Screw_Terminal_01x06
Connections:
- net GND: now also J19.6 (Pin_6)
Changed lines of the file:
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@@
+	)
+	(symbol
+		(lib_id "power:GND")
+		(at 34.29 151.13 0)
+		(unit 1)
+		(exclude_from_sim no)
+		(in_bom yes)
+		(on_board yes)
+		(dnp no)
+		(fields_autoplaced yes)
+		(property "Reference" "#PWR0244"
+			(at 34.29 157.48 0)
+			(effects
+				(font
+					(size 1.27 1.27)
+				)
+				(hide yes)
+			)
+		)
+		(property "Value" "GND"
+			(at 34.29 156.21 0)
+			(effects
+				(font
+					(size 1.27 1.27)
+				)
+			)
+		)
+		(property "Footprint" ""
+			(at 34.29 151.13 0)
+			(effects
+				(font
+					(size 1.27 1.27)
+				)
+				(hide yes)
+			)
+		)
+		(property "Datasheet" ""
+			(at 34.29 151.13 0)
+			(effects
+				(font
+					(size 1.27 1.27)
+				)
+				(hide yes)
+			)
+		)
+		(property "Description" "Power symbol creates a global label with name \"GND\" , ground"
+			(at 34.29 151.13 0)
+			(effects
+				(font
+					(size 1.27 1.27)
+				)
+				(hide yes)
+			)
+		)
+		(pin "1"
+		)
+		(instances
+			(project "Console"
+				(path "/10b20c6b-8045-46d1-a965-0d7dd9a1b5fa/00000000-0000-0000-0000-0000560f49b9"
+					(reference "#PWR0244")
+					(unit 1)
+				)
+			)
+		)
 	)
 	(symbol
@@
 	)
 	(symbol
-		(lib_id "Connector:Screw_Terminal_01x05")
+		(lib_id "Connector:Screw_Terminal_01x06")
 		(at 39.37 143.51 0)
 		(unit 1)
@@
 		(fields_autoplaced yes)
 		(property "Reference" "J19"
-			(at 41.91 142.2399 0)
-			(effects
-				(font
-					(size 1.27 1.27)
-				)
-				(justify left)
-			)
-		)
-		(property "Value" "Screw_Terminal_01x05"
-			(at 41.91 144.7799 0)
-			(effects
-				(font
-					(size 1.27 1.27)
-				)
-				(justify left)
-			)
-		)
-		(property "Footprint" "TerminalBlock_RND:TerminalBlock_RND_205-00004_1x05_P5.00mm_Horizontal"
+			(at 41.91 143.5099 0)
+			(effects
+				(font
+					(size 1.27 1.27)
+				)
+				(justify left)
+			)
+		)
+		(property "Value" "Screw_Terminal_01x06"
+			(at 41.91 146.0499 0)
+			(effects
+				(font
+					(size 1.27 1.27)
+				)
+				(justify left)
+			)
+		)
+		(property "Footprint" "TerminalBlock_RND:TerminalBlock_RND_205-00005_1x06_P5.00mm_Horizontal"
 			(at 39.37 143.51 0)
 			(effects
@@
 			)
 		)
-		(property "Description" "Generic screw terminal, single row, 01x05, script generated (kicad-library-utils/schlib/autogen/connector/)"
+		(property "Description" "Generic screw terminal, single row, 01x06, script generated (kicad-library-utils/schlib/autogen/connector/)"
 			(at 39.37 143.51 0)
 			(effects
@@
 		(pin "3"
 		)
-		(instances
+		(pin "6"
+		)
+		(instances
